Commit message: completed

File: src/description/urdf/gazebo.urdf (robot description, URDF)
Before this commit: robot E1, 17 links, 16 joints
Links:
- link ankle_l: mass None -> 1.0; geometry collision cylinder length=0.5 radius=0.2; visual cylinder length=0.5 radius=0.15
- link ankle_lower_l: mass None -> 1.0; geometry collision cylinder length=0.5 radius=0.2; visual cylinder length=0.55 radius=0.15
- link ankle_lower_r: mass None -> 1.0; geometry collision cylinder length=0.5 radius=0.2; visual cylinder length=0.55 radius=0.15
- link ankle_r: mass None -> 1.0; geometry collision cylinder length=0.5 radius=0.2; visual cylinder length=0.5 radius=0.15
- link body: mass None -> 1.0; geometry collision box size=1 1.5 1; visual box size=1 1.5 1
- link foot_l: mass None -> 1.0; geometry collision cylinder length=0.5 radius=0.2; visual cylinder length=0.7 radius=0.15
- link foot_r: mass None -> 1.0; geometry collision cylinder length=0.5 radius=0.2; visual cylinder length=0.7 radius=0.15
- link hip_l: mass None -> 1.0; geometry collision cylinder length=0.5 radius=0.2; visual cylinder length=0.5 radius=0.2
- link hip_r: mass None -> 1.0; geometry collision cylinder length=0.5 radius=0.2; visual cylinder length=0.5 radius=0.2
- link knee_l: mass None -> 1.0; geometry collision cylinder length=0.5 radius=0.2; visual cylinder length=0.55 radius=0.2
- link knee_r: mass None -> 1.0; geometry collision cylinder length=0.5 radius=0.2; visual cylinder length=0.55 radius=0.2
- link leg_l: mass None -> 1.0; geometry collision cylinder length=0.5 radius=0.2; visual cylinder length=0.7 radius=0.15
- link leg_r: mass None -> 1.0; geometry collision cylinder length=0.5 radius=0.2; visual cylinder length=0.7 radius=0.15
- link lower_hip_l: mass None -> 1.0; geometry collision cylinder length=0.5 radius=0.2; visual cylinder length=0.5 radius=0.2
- link lower_hip_r: mass None -> 1.0; geometry collision cylinder length=0.5 radius=0.2; visual cylinder length=0.5 radius=0.2
- link toe_l: mass None -> 1.0; geometry collision cylinder length=0.5 radius=0.2; visual box size=0.6 0.2 0.9
- link toe_r: mass None -> 1.0; geometry collision cylinder length=0.5 radius=0.2; visual box size=0.6 0.2 0.9
