Commit message: done

File: src/description/urdf/robot_E1.xacro (robot description, xacro)
@@ -1,4 +1,14 @@
 <?xml version="1.0" ?>
 <robot name="Asimo_E1" xmlns:xacro="http://www.ros.org/wiki/xacro">
+  <!-- Constants value-->
+  <xacro:property name="PI" value="3.1415926535897931"/>
+  <!-- color-->
+  <material name="white">
+        <color rgba="1 1 1 1"/>
+  </material>
+  <material name="red">
+    <color rgba="1 0 0 1"/>
+  </material>
+  <!-- Link Joint Description-->
   <link name="body">
     <visual>
@@ -7,23 +17,23 @@
         <box size="1 1.5 1"/>
       </geometry>
-      <material name="white">
-        <color rgba="1 1 1 1"/>
-      </material>
+      <material name="white"/>
     </visual>
   </link>
   <link name="hip_l">
     <visual>
-      <origin rpy="1.57075 0 1.57075" xyz="0 -0.5 -1.2"/>
-      <geometry>
-        <cylinder length="0.5" radius="0.2"/>
-      </geometry>
+      <origin rpy="${PI/2} 0 ${PI/2}" xyz="0 -0.5 -1.2"/>
+      <geometry>
+        <cylinder length="0.5" radius="0.2"/>
+      </geometry>
+      <material name="red"/>
     </visual>
   </link>
   <link name="hip_r">
     <visual>
-      <origin rpy="1.57075 0 1.57075" xyz="0 0.5 -1.2"/>
-      <geometry>
-        <cylinder length="0.5" radius="0.2"/>
-      </geometry>
+      <origin rpy="${PI/2}  0 ${PI/2}" xyz="0 0.5 -1.2"/>
+      <geometry>
+        <cylinder length="0.5" radius="0.2"/>
+      </geometry>
+      <material name="red"/>
     </visual>
   </link>
@@ -38,16 +48,18 @@
   <link name="lower_hip_r">
     <visual>
-      <origin rpy="1.57075 0 0" xyz="0 0.5 -1.5"/>
-      <geometry>
-        <cylinder length="0.5" radius="0.2"/>
-      </geometry>
+      <origin rpy="${PI/2} 0 0" xyz="0 0.5 -1.5"/>
+      <geometry>
+        <cylinder length="0.5" radius="0.2"/>
+      </geometry>
+      <material name="red"/>
     </visual>
   </link>
   <link name="lower_hip_l">
     <visual>
-      <origin rpy="1.57075 0 0" xyz="0 -0.5 -1.5"/>
-      <geometry>
-        <cylinder length="0.5" radius="0.2"/>
-      </geometry>
+      <origin rpy="${PI/2} 0 0" xyz="0 -0.5 -1.5"/>
+      <geometry>
+        <cylinder length="0.5" radius="0.2"/>
+      </geometry>
+      <material name="red"/>
     </visual>
   </link>
@@ -62,22 +74,18 @@
   <link name="leg_l">
     <visual>
-      <origin rpy="0 0 1.57075" xyz="0 -0.5 -2"/>
-      <geometry>
-        <cylinder length="0.7" radius="0.15"/>
-      </geometry>
-      <material name="white">
-        <color rgba="1 1 1 1"/>
-      </material>
+      <origin rpy="0 0 ${PI/2}" xyz="0 -0.5 -2"/>
+      <geometry>
+        <cylinder length="0.7" radius="0.15"/>
+      </geometry>
+      <material name="white"/>
     </visual>
   </link>
   <link name="leg_r">
     <visual>
-      <origin rpy="0 0 1.57075" xyz="0 0.5 -2"/>
-      <geometry>
-        <cylinder length="0.7" radius="0.15"/>
-      </geometry>
-      <material name="white">
-        <color rgba="1 1 1 1"/>
-      </material>
+      <origin rpy="0 0 ${PI/2}" xyz="0 0.5 -2"/>
+      <geometry>
+        <cylinder length="0.7" radius="0.15"/>
+      </geometry>
+      <material name="white"/>
     </visual>
   </link>
@@ -92,13 +100,14 @@
   <link name="knee_r">
     <visual>
-      <origin rpy="1.57075 0 0" xyz="0 0.5 -2.5"/>
+      <origin rpy="${PI/2} 0 0" xyz="0 0.5 -2.5"/>
       <geometry>
         <cylinder length="0.55" radius="0.2"/>
       </geometry>
+      <material name="red"/>
     </visual>
   </link>
   <link name="knee_l">
     <visual>
-      <origin rpy="1.57075 0 0" xyz="0 -0.5 -2.5"/>
+      <origin rpy="${PI/2} 0 0" xyz="0 -0.5 -2.5"/>
       <geometry>
         <cylinder length="0.55" radius="0.2"/>
@@ -116,22 +125,18 @@
   <link name="foot_l">
     <visual>
-      <origin rpy="0 0 1.57075" xyz="0 -0.5 -3"/>
-      <geometry>
-        <cylinder length="0.7" radius="0.15"/>
-      </geometry>
-        <material name="white">
-        <color rgba="1 1 1 1"/>
-      </material>
+      <origin rpy="0 0 ${PI/2}" xyz="0 -0.5 -3"/>
+      <geometry>
+        <cylinder length="0.7" radius="0.15"/>
+      </geometry>
+      <material name="white"/>
     </visual>
   </link>
   <link name="foot_r">
     <visual>
-      <origin rpy="0 0 1.57075" xyz="0 0.5 -3"/>
-      <geometry>
-        <cylinder length="0.7" radius="0.15"/>
-      </geometry>
-        <material name="white">
-        <color rgba="1 1 1 1"/>
-      </material>
+      <origin rpy="0 0 ${PI/2}" xyz="0 0.5 -3"/>
+      <geometry>
+        <cylinder length="0.7" radius="0.15"/>
+      </geometry>
+        <material name="white"/>
     </visual>
   </link>
@@ -146,16 +151,18 @@
   <link name="ankle_l">
     <visual>
-      <origin rpy="1.57075 0 0" xyz="0 -0.5 -3.5"/>
+      <origin rpy="${PI/2} 0 0" xyz="0 -0.5 -3.5"/>
       <geometry>
         <cylinder length="0.5" radius="0.15"/>
       </geometry>
+      <material name="red"/>
     </visual>
   </link>
   <link name="ankle_r">
     <visual>
-      <origin rpy="1.57075 0 0" xyz="0 0.5 -3.5"/>
+      <origin rpy="${PI/2} 0 0" xyz="0 0.5 -3.5"/>
       <geometry>
         <cylinder length="0.5" radius="0.15"/>
       </geometry>
+      <material name="red"/>
     </visual>
   </link>
@@ -170,16 +177,18 @@
   <link name="ankle_lower_l">
     <visual>
-      <origin rpy="1.57075 0 1.57075" xyz="0 -0.5 -3.7"/>
+      <origin rpy="${PI/2} 0 ${PI/2}" xyz="0 -0.5 -3.7"/>
       <geometry>
         <cylinder length="0.55" radius="0.15"/>
       </geometry>
+      <material name="red"/>
     </visual>
   </link>
   <link name="ankle_lower_r">
     <visual>
-      <origin rpy="1.57075 0 1.57075" xyz="0 0.5 -3.7"/>
+      <origin rpy="${PI/2} 0 ${PI/2}" xyz="0 0.5 -3.7"/>
       <geometry>
         <cylinder length="0.55" radius="0.15"/>
       </geometry>
+      <material name="red"/>
     </visual>
   </link>
@@ -194,22 +203,18 @@
   <link name="toe_r">
     <visual>
-      <origin rpy="1.57075 0 1.57075" xyz="0.1 0.5 -3.9"/>
+      <origin rpy="${PI/2} 0 ${PI/2}" xyz="0.1 0.5 -3.9"/>
       <geometry>
         <box size="0.6 0.2 0.9"/>
       </geometry>
-        <material name="white">
-        <color rgba="1 1 1 1"/>
-      </material>
+        <material name="white"/>
     </visual>
   </link>
   <link name="toe_l">
     <visual>
-      <origin rpy="1.57075 0 1.57075" xyz="0.1 -0.5 -3.9"/>
+      <origin rpy="${PI/2} 0 ${PI/2}" xyz="0.1 -0.5 -3.9"/>
       <geometry>
         <box size="0.6 0.2 0.9"/>
       </geometry>
-        <material name="white">
-        <color rgba="1 1 1 1"/>
-      </material>
+        <material name="white"/>
     </visual>
   </link>
