Commit message: add script to take photo

File: src/asimo_e1_description/urdf/links_joints.xacro (robot description, xacro)
@@ -78,4 +78,24 @@
     </link>
   </xacro:macro>
+  <!-- Hokuyo Laser -->
+  <link name="hokuyo">
+    <collision>
+      <origin xyz="0 0 0" rpy="0 0 0"/>
+      <geometry>
+    <box size="0.1 0.1 0.1"/>
+      </geometry>
+    </collision>
+    <visual>
+      <origin xyz="0 0 0" rpy="0 0 0"/>
+      <geometry>
+        <mesh filename="package://asimo_e1_description/meshes/hokuyo.dae"/>
+      </geometry>
+    </visual>
+    <inertial>
+      <mass value="1e-5" />
+      <origin xyz="0 0 0" rpy="0 0 0"/>
+      <inertia ixx="1e-6" ixy="0" ixz="0" iyy="1e-6" iyz="0" izz="1e-6" />
+    </inertial>
+  </link>
   <!-- <material name="black">
     <color rgba="0.0 0.0 0.0 1.0"/>

File: src/asimo_e1_description/urdf/robot_E1_v2.xacro (robot description, xacro)
@@ -20,4 +20,19 @@
                 origin_rpy="0 0 0" origin_xyz="0.5 0 3.4"
                 parent="body" child="camera"/>
+  <!-- Hokuyo Laser -->
+<!-- <link_box name="hokuyo"
+              origin_rpy="0 0 0" origin_xyz="0 0 0"
+              mass="${cameraMass}"
+              ixx="1e-7" ixy="0" ixz="0" iyy="1e-7" iyz="0" izz="1e-7"
+              size="${cameraSize} ${cameraSize} ${cameraSize}"
+              color = 'red'
+               <geometry>
+        <mesh filename="package://asimo_e1_description/meshes/hokuyo.dae"/>
+      </geometry>
+      /> -->
+<fixed_joint name="hokuyo_joint" type="fixed"
+                axis_xyz="0 1 0"
+                origin_rpy="0 0 0" origin_xyz="0.5 0 4"
+                parent="body" child="hokuyo"/>
 <!-- <link name="dummy">
    </link>
@@ -275,3 +290,39 @@
     </sensor>
   </gazebo>
+    <!-- hokuyo -->
+  <gazebo reference="hokuyo">
+    <sensor type="gpu_ray" name="head_hokuyo_sensor">
+      <pose>0 0 0 0 0 0</pose>
+      <visualize>true</visualize>
+      <update_rate>40</update_rate>
+      <ray>
+        <scan>
+          <horizontal>
+            <samples>720</samples>
+            <resolution>1</resolution>
+            <min_angle>-1.570796</min_angle>
+            <max_angle>1.570796</max_angle>
+          </horizontal>
+        </scan>
+        <range>
+          <min>15</min>
+          <max>30.0</max>
+          <resolution>0.01</resolution>
+        </range>
+        <noise>
+          <type>gaussian</type>
+          <!-- Noise parameters based on published spec for Hokuyo laser
+               achieving "+-30mm" accuracy at range < 10m.  A mean of 0.0m and
+               stddev of 0.01m will put 99.7% of samples within 0.03m of the true
+               reading. -->
+          <mean>0.0</mean>
+          <stddev>0.01</stddev>
+        </noise>
+      </ray>
+      <plugin name="gazebo_ros_head_hokuyo_controller" filename="libgazebo_ros_gpu_laser.so">
+        <topicName>/mybot/laser/scan</topicName>
+        <frameName>hokuyo</frameName>
+      </plugin>
+    </sensor>
+  </gazebo>
 </robot>

Commit message: add color and world in gazebo

File: src/asimo_e1_description/urdf/links_joints.xacro (robot description, xacro)
@@ -1,10 +1,4 @@
 <?xml version="1.0" ?>
 <robot xmlns:xacro="http://www.ros.org/wiki/xacro">
-  <material name="white">
-    <color rgba="1 1 1 1"/>
-  </material>
-  <material name="red">
-    <color rgba="1 0 0 1"/>
-  </material>
   <xacro:macro name="rot_joint" params="name type axis_xyz origin_rpy origin_xyz parent child limit_e limit_l limit_u limit_v">
     <joint name="${name}" type="${type}">
@@ -98,5 +92,6 @@
     </inertial>
   </link>
-  <!-- <material name="black">
+<!-- Color -->
+ <material name="black">
     <color rgba="0.0 0.0 0.0 1.0"/>
   </material>
@@ -107,12 +102,18 @@
     <color rgba="0.0 0.8 0.0 1.0"/>
   </material>
-  <material name="gray">
-    <color rgba="0.7 0.7 0.7 1.0"/>
+  <material name="grey">
+    <color rgba="0.2 0.2 0.2 1.0"/>
   </material>
-  <material name="darkgray">
-    <color rgba="0.3 0.3 0.3 1.0"/>
+  <material name="orange">
+    <color rgba="${255/255} ${108/255} ${10/255} 1.0"/>
   </material>
-  <material name="yellow">
-    <color rgba="0.8 0.8 0.0 1.0"/>
-  </material> -->
+  <material name="brown">
+    <color rgba="${222/255} ${207/255} ${195/255} 1.0"/>
+  </material>
+  <material name="red">
+    <color rgba="0.8 0.0 0.0 1.0"/>
+  </material>
+  <material name="white">
+    <color rgba="1.0 1.0 1.0 1.0"/>
+  </material>
 </robot>

File: src/asimo_e1_description/urdf/robot_E1_v2.xacro (robot description, xacro)
@@ -23,5 +23,5 @@
 <fixed_joint name="hokuyo_joint" type="fixed"
                 axis_xyz="0 1 0"
-                origin_rpy="0 0 0" origin_xyz="0.5 0 4"
+                origin_rpy="0 0 0" origin_xyz="0.5 0 3.9"
                 parent="body" child="hokuyo"/>
 <!-- <link name="dummy">
@@ -38,5 +38,5 @@
               izz="170.667"
               size="1 1.5 1"
-              color = 'white' />
+              color = 'orange' />
  <link_cylinder name="hip_l"
               origin_rpy="${PI/2}  0 ${PI/2}" origin_xyz="0 0 0"
